File: DC-DC Boost Converter.kicad_sch (KiCad schematic)
At the start: 0 parts

Commit message: Added External Symbol xl6009
Other:
- title: (none) -> DC-DC Boost Converter
Changed lines of the file:
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@@
 	(generator_version "9.0")
 	(paper "A4")
+	(title_block
+		(title "DC-DC Boost Converter")
+	)
 	(sheet_instances
 		(path "/"

Commit message: Added all the Components to Schematic Editor
Parts:
- added C1, C2, C3, C4: C, symbol Device:C
- added D1: SS34, Diode_SMD:D_SMA, symbol Diode:SS34
- added J1, J2, J3, J4: Conn_01x01_Pin, symbol Connector:Conn_01x01_Pin
- added L1: L, symbol Device:L
- added R1: R, symbol Device:R
- added RV1: R_Potentiometer, symbol Device:R_Potentiometer
- added VR1: XL6009, XL6009:DPAK170P1435X465-6N, symbol XL6009:XL6009
Connections:
- new net: VR1.3 (SW), VR1.6 (SW)
